File: project2.kicad_sch (KiCad schematic)
At the start: 15 parts, among them J1 USB_C_Receptacle_PowerOnly_6P, Q1 FS8205A, Q2 DW01A, U1 TP4056-42-ESOP8

Commit message: MT3608 added
Parts:
- added C3, C4: C, Diode_SMD:D_SMA, symbol Device:C
- added D3: SS34, Diode_SMD:D_SMA, symbol Diode:SS34
- added J2, J3, J4, J5: Conn_01x01_Socket, Connector_Wire:SolderWirePad_1x01_SMD_1.5x3mm, symbol Connector:Conn_01x01_Socket
- added L1: 22uH, Inductor_SMD:L_7.3x7.3_H4.5, symbol Device:L
- added R10: 16k, Resistor_SMD:R_0805_2012Metric, symbol Device:R
- added R8: 2.2k, Resistor_SMD:R_0805_2012Metric, symbol Device:R
- added R9: 42k, Resistor_SMD:R_0805_2012Metric, symbol Device:R
- added SW1: SW_Nidec_CAS-120A1, Button_Switch_SMD:Nidec_Copal_CAS-120A, symbol Switch:SW_Nidec_CAS-120A1
- added U2: MT3608, Package_TO_SOT_SMD:SOT-23-6, symbol Regulator_Switching:MT3608
Connections:
- net BAT+: now also C3.1, J5.1 (Pin_1), L1.1, U2.4 (EN), U2.5 (IN)
- net GND: now also C3.2, C4.1, J3.1 (Pin_1), J4.1 (Pin_1), R8.2, U2.2 (GND)
- new net: D3.2 (A), L1.2, U2.1 (SW)
- new net: R10.1, R8.1, R9.1, U2.3 (FB)
- new net: R9.2, SW1.1 (C)
- new net: R10.2, SW1.3 (A)
- new net OUT+: C4.2, D3.1 (K), J2.1 (Pin_1), SW1.2 (B)
Other:
- moved on the sheet: C1, C2, D1, D2, J1, Q1, R1, R2, R3, R4, R5, R6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

Commit message: PCB created
Other:
- note added: "5V / 12V DUAL-OUTPUT BOOST CONVERTER (MT3608)"
- note added: "SYSTEM OUTPUT \& BATTERY TERMINALS"
- note added: "USB-C CHARGER \& BATTERY PROTECTION (TP4056 + DW01A)"
- company: (none) -> Devendra Kashyap
- title: (none) -> Li-Po Battery Charger & Selectable 5V/12V Boost Module
- moved on the sheet: C1, C2, C3, C4, D1, D2, D3, J1, J2, J3, J4, J5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
